File: board/kicad/mega_videl/ddr3power.kicad_sch (KiCad schematic)
At the start: 45 parts, among them U1 TPS51200DRCR

Commit message: Reviewed and fixed many issues. e.g. missing decoupling for 1.35v under fpga
Parts:
- renumbered C52 to C51, C53 to C52, C54 to C53, C55 to C54, C56 to C55, C57 to C56, C58 to C57, C59 to C58, C60 to C59, C61 to C60, C62 to C61, C63 to C62, C64 to C63, C65 to C64, C66 to C65, C67 to C66, C68 to C67, C69 to C68, C70 to C69, C71 to C70, C72 to C71, C73 to C72, C74 to C73, C75 to C74, C76 to C75, C77 to C76
Connections:
- net +1V35: now also C11.1, C12.1, U1.2 (VLDOIN)
- net +3V3: no longer C11.1, C12.1, U1.2 (VLDOIN)
Changed lines of the file:
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@@
 	)
 	(junction
-		(at 80.01 123.19)
-		(diameter 0)
-		(color 0 0 0 0)
-	)
-	(junction
 		(at 59.69 152.4)
 		(diameter 0)
@@
 	)
 	(junction
-		(at 113.03 109.22)
-		(diameter 0)
-		(color 0 0 0 0)
-	)
-	(junction
 		(at 66.04 152.4)
 		(diameter 0)
@@
 	)
 	(junction
+		(at 68.58 123.19)
+		(diameter 0)
+		(color 0 0 0 0)
+	)
+	(junction
 		(at 214.63 46.99)
 		(diameter 0)
@@
 	)
 	(junction
+		(at 80.01 123.19)
+		(diameter 0)
+		(color 0 0 0 0)
+	)
+	(junction
 		(at 96.52 142.24)
 		(diameter 0)
@@
 	(wire
 		(pts
-			(xy 80.01 109.22) (xy 80.01 123.19)
-		)
-		(stroke
-			(width 0)
-			(type default)
-		)
-	)
-	(wire
-		(pts
 			(xy 132.08 142.24) (xy 138.43 142.24)
 		)
@@
 	(wire
 		(pts
+			(xy 68.58 123.19) (xy 80.01 123.19)
+		)
+		(stroke
+			(width 0)
+			(type default)
+		)
+	)
+	(wire
+		(pts
 			(xy 27.94 83.82) (xy 36.83 83.82)
 		)
@@
 	(wire
 		(pts
-			(xy 80.01 109.22) (xy 113.03 109.22)
-		)
-		(stroke
-			(width 0)
-			(type default)
-		)
-	)
-	(wire
-		(pts
 			(xy 113.03 142.24) (xy 132.08 142.24)
 		)
@@
 		(in_pos_files yes)
 		(dnp no)
-		(property "Reference" "C68"
+		(property "Reference" "C67"
 			(at 117.348 42.164 0)
 			(show_name no)
@@
 			(project "mega_videl"
 				(path "/10511203-7d65-4cdf-a1a4-c07b44ea87e2/cdbe408a-30b2-43ec-8cff-a9bfdb2a9228"
-					(reference "C68")
+					(reference "C67")
 					(unit 1)
 				)
@@
 		(in_pos_files yes)
 		(dnp no)
-		(property "Reference" "C67"
+		(property "Reference" "C66"
 			(at 120.396 88.138 0)
 			(show_name no)
@@
 			(project "mega_videl"
 				(path "/10511203-7d65-4cdf-a1a4-c07b44ea87e2/cdbe408a-30b2-43ec-8cff-a9bfdb2a9228"
-					(reference "C67")
+					(reference "C66")
 					(unit 1)
 				)
@@
 		(in_pos_files yes)
 		(dnp no)
-		(property "Reference" "C55"
+		(property "Reference" "C54"
 			(at 51.308 40.894 0)
 			(show_name no)
@@
 			(project "mega_videl"
 				(path "/10511203-7d65-4cdf-a1a4-c07b44ea87e2/cdbe408a-30b2-43ec-8cff-a9bfdb2a9228"
-					(reference "C55")
+					(reference "C54")
 					(unit 1)
 				)
@@
 		(in_pos_files yes)
 		(dnp no)
-		(property "Reference" "C54"
+		(property "Reference" "C53"
 			(at 42.418 40.894 0)
 			(show_name no)
@@
 			(project "mega_videl"
 				(path "/10511203-7d65-4cdf-a1a4-c07b44ea87e2/cdbe408a-30b2-43ec-8cff-a9bfdb2a9228"
-					(reference "C54")
+					(reference "C53")
 					(unit 1)
 				)
@@
 		(in_pos_files yes)
 		(dnp no)
-		(property "Reference" "C72"
+		(property "Reference" "C71"
 			(at 130.556 88.138 0)
 			(show_name no)
@@
 			(project "mega_videl"
 				(path "/10511203-7d65-4cdf-a1a4-c07b44ea87e2/cdbe408a-30b2-43ec-8cff-a9bfdb2a9228"
-					(reference "C72")
+					(reference "C71")
 					(unit 1)
 				)
@@
 		(in_pos_files yes)
 		(dnp no)
-		(property "Reference" "C66"
+		(property "Reference" "C65"
 			(at 127.508 42.164 0)
 			(show_name no)
@@
 			(project "mega_videl"
 				(path "/10511203-7d65-4cdf-a1a4-c07b44ea87e2/cdbe408a-30b2-43ec-8cff-a9bfdb2a9228"
-					(reference "C66")
+					(reference "C65")
 					(unit 1)
 				)
@@
 		(in_pos_files yes)
 		(dnp no)
-		(property "Reference" "C73"
+		(property "Reference" "C72"
 			(at 89.408 42.164 0)
 			(show_name no)
@@
 			(project "mega_videl"
 				(path "/10511203-7d65-4cdf-a1a4-c07b44ea87e2/cdbe408a-30b2-43ec-8cff-a9bfdb2a9228"
-					(reference "C73")
+					(reference "C72")
 					(unit 1)
 				)
@@
 		(in_pos_files yes)
 		(dnp no)
-		(property "Reference" "C59"
+		(property "Reference" "C58"
 			(at 63.246 88.138 0)
 			(show_name no)
@@
 			(project "mega_videl"
 				(path "/10511203-7d65-4cdf-a1a4-c07b44ea87e2/cdbe408a-30b2-43ec-8cff-a9bfdb2a9228"
-					(reference "C59")
+					(reference "C58")
 					(unit 1)
 				)
@@
 		(dnp no)
 		(fields_autoplaced yes)
-		(property "Reference" "C61"
+		(property "Reference" "C60"
 			(at 31.75 110.4899 0)
 			(show_name no)
@@
 			(project "mega_videl"
 				(path "/10511203-7d65-4cdf-a1a4-c07b44ea87e2/cdbe408a-30b2-43ec-8cff-a9bfdb2a9228"
-					(reference "C61")
+					(reference "C60")
 					(unit 1)
 				)
@@
 		(in_pos_files yes)
 		(dnp no)
-		(property "Reference" "C77"
+		(property "Reference" "C76"
 			(at 36.576 86.868 0)
 			(show_name no)
@@
 			(project "mega_videl"
 				(path "/10511203-7d65-4cdf-a1a4-c07b44ea87e2/cdbe408a-30b2-43ec-8cff-a9bfdb2a9228"
-					(reference "C77")
+					(reference "C76")
 					(unit 1)
 				)
@@
 		(in_pos_files yes)
 		(dnp no)
-		(property "Reference" "C65"
+		(property "Reference" "C64"
 			(at 92.456 88.138 0)
 			(show_name no)
@@
 			(project "mega_videl"
 				(path "/10511203-7d65-4cdf-a1a4-c07b44ea87e2/cdbe408a-30b2-43ec-8cff-a9bfdb2a9228"
-					(reference "C65")
+					(reference "C64")
 					(unit 1)
 				)
@@
 		(dnp no)
 		(fields_autoplaced yes)
-		(property "Reference" "C62"
+		(property "Reference" "C61"
 			(at 41.91 110.4899 0)
 			(hide yes)
@@
 			(project "mega_videl"
 				(path "/10511203-7d65-4cdf-a1a4-c07b44ea87e2/cdbe408a-30b2-43ec-8cff-a9bfdb2a9228"
-					(reference "C62")
+					(reference "C61")
 					(unit 1)
 				)
@@
 		(in_pos_files yes)
 		(dnp no)
-		(property "Reference" "C69"
+		(property "Reference" "C68"
 			(at 79.248 42.164 0)
 			(show_name no)
@@
 			(project "mega_videl"
 				(path "/10511203-7d65-4cdf-a1a4-c07b44ea87e2/cdbe408a-30b2-43ec-8cff-a9bfdb2a9228"
-					(reference "C69")
+					(reference "C68")
 					(unit 1)
 				)
@@
 		(in_pos_files yes)
 		(dnp no)
-		(property "Reference" "C64"
+		(property "Reference" "C63"
 			(at 98.298 42.164 0)
 			(show_name no)
@@
 			(project "mega_videl"
 				(path "/10511203-7d65-4cdf-a1a4-c07b44ea87e2/cdbe408a-30b2-43ec-8cff-a9bfdb2a9228"
-					(reference "C64")
+					(reference "C63")
 					(unit 1)
 				)
@@
 		(in_pos_files yes)
 		(dnp no)
-		(property "Reference" "C53"
+		(property "Reference" "C52"
 			(at 54.356 86.868 0)
 			(show_name no)
@@
 			(project "mega_videl"
 				(path "/10511203-7d65-4cdf-a1a4-c07b44ea87e2/cdbe408a-30b2-43ec-8cff-a9bfdb2a9228"
-					(reference "C53")
+					(reference "C52")
 					(unit 1)
 				)
@@
 		(in_pos_files yes)
 		(dnp no)
-		(property "Reference" "C57"
+		(property "Reference" "C56"
 			(at 82.296 88.138 0)
 			(show_name no)
@@
 			(project "mega_videl"
 				(path "/10511203-7d65-4cdf-a1a4-c07b44ea87e2/cdbe408a-30b2-43ec-8cff-a9bfdb2a9228"
-					(reference "C57")
+					(reference "C56")
 					(unit 1)
 				)
@@
 		(in_pos_files yes)
 		(dnp no)
-		(property "Reference" "C52"
+		(property "Reference" "C51"
 			(at 27.686 86.868 0)
 			(show_name no)
@@
 			(project "mega_videl"
 				(path "/10511203-7d65-4cdf-a1a4-c07b44ea87e2/cdbe408a-30b2-43ec-8cff-a9bfdb2a9228"
-					(reference "C52")
+					(reference "C51")
 					(unit 1)
 				)
@@
 		(in_pos_files yes)
 		(dnp no)
-		(property "Reference" "C56"
+		(property "Reference" "C55"
 			(at 60.198 42.164 0)
 			(show_name no)
@@
 			(project "mega_videl"
 				(path "/10511203-7d65-4cdf-a1a4-c07b44ea87e2/cdbe408a-30b2-43ec-8cff-a9bfdb2a9228"
-					(reference "C56")
+					(reference "C55")
 					(unit 1)
 				)
@@
 		(in_pos_files yes)
 		(dnp no)
-		(property "Reference" "C76"
+		(property "Reference" "C75"
 			(at 45.466 86.868 0)
 			(show_name no)
@@
 			(project "mega_videl"
 				(path "/10511203-7d65-4cdf-a1a4-c07b44ea87e2/cdbe408a-30b2-43ec-8cff-a9bfdb2a9228"
-					(reference "C76")
+					(reference "C75")
 					(unit 1)
 				)
@@
 		(in_pos_files yes)
 		(dnp no)
-		(property "Reference" "C71"
+		(property "Reference" "C70"
 			(at 72.136 88.138 0)
 			(show_name no)
@@
 			(project "mega_videl"
 				(path "/10511203-7d65-4cdf-a1a4-c07b44ea87e2/cdbe408a-30b2-43ec-8cff-a9bfdb2a9228"
-					(reference "C71")
+					(reference "C70")
 					(unit 1)
 				)
@@
 		(in_pos_files yes)
 		(dnp no)
-		(property "Reference" "C74"
+		(property "Reference" "C73"
 			(at 24.638 40.894 0)
 			(show_name no)
@@
 			(project "mega_videl"
 				(path "/10511203-7d65-4cdf-a1a4-c07b44ea87e2/cdbe408a-30b2-43ec-8cff-a9bfdb2a9228"
-					(reference "C74")
+					(reference "C73")
 					(unit 1)
 				)
@@
 		(in_pos_files yes)
 		(dnp no)
-		(property "Reference" "C75"
+		(property "Reference" "C74"
 			(at 33.528 40.894 0)
 			(show_name no)
@@
 			(project "mega_videl"
 				(path "/10511203-7d65-4cdf-a1a4-c07b44ea87e2/cdbe408a-30b2-43ec-8cff-a9bfdb2a9228"
-					(reference "C75")
+					(reference "C74")
 					(unit 1)
 				)
@@
 		(in_pos_files yes)
 		(dnp no)
-		(property "Reference" "C58"
+		(property "Reference" "C57"
 			(at 107.188 42.164 0)
 			(show_name no)
@@
 			(project "mega_videl"
 				(path "/10511203-7d65-4cdf-a1a4-c07b44ea87e2/cdbe408a-30b2-43ec-8cff-a9bfdb2a9228"
-					(reference "C58")
+					(reference "C57")
 					(unit 1)
 				)
@@
 		(in_pos_files yes)
 		(dnp no)
-		(property "Reference" "C63"
+		(property "Reference" "C62"
 			(at 110.236 88.138 0)
 			(show_name no)
@@
 			(project "mega_videl"
 				(path "/10511203-7d65-4cdf-a1a4-c07b44ea87e2/cdbe408a-30b2-43ec-8cff-a9bfdb2a9228"
-					(reference "C63")
+					(reference "C62")
 					(unit 1)
 				)
@@
 		(in_pos_files yes)
 		(dnp no)
-		(property "Reference" "C60"
+		(property "Reference" "C59"
 			(at 101.346 88.138 0)
 			(show_name no)
@@
 			(project "mega_videl"
 				(path "/10511203-7d65-4cdf-a1a4-c07b44ea87e2/cdbe408a-30b2-43ec-8cff-a9bfdb2a9228"
-					(reference "C60")
+					(reference "C59")
 					(unit 1)
 				)
@@
 		(in_pos_files yes)
 		(dnp no)
-		(property "Reference" "C70"
+		(property "Reference" "C69"
 			(at 69.088 42.164 0)
 			(show_name no)
@@
 			(project "mega_videl"
 				(path "/10511203-7d65-4cdf-a1a4-c07b44ea87e2/cdbe408a-30b2-43ec-8cff-a9bfdb2a9228"
-					(reference "C70")
+					(reference "C69")
 					(unit 1)
 				)

Commit message: Assigned all parts with JLCPCB plugin
Parts:
- C1, C60, C61: LCSC (none) -> C14663
- C10: LCSC (none) -> C1588
- C11, C12, C2, C3, C5, C6, C7: LCSC (none) -> C15850
- C4, C51, C52, C53, C54, C73, C74, C75, C76: LCSC (none) -> C1779
- C55, C56, C57, C58, C59, C62, C63, C64, C65, C66, C67, C68, C69, C70, C71, C72: LCSC (none) -> C1525
- R1, R2: LCSC (none) -> C25804
