File: board/kicad/mega_videl/PCIe.kicad_sch (KiCad schematic)
At the start: 14 parts, among them U13 PI6CG33201CZDIEX, U16 HC-USB3.0-L168-WP, Y2 25MHz

Commit message: Reviewed and fixed many issues. e.g. missing decoupling for 1.35v under fpga
Parts:
- added C115, C116, C121: 0.1uF, Capacitor_SMD:C_0402_1005Metric, symbol Device:C
- added C120: 4.7uF, Capacitor_SMD:C_0805_2012Metric, symbol Device:C
- C122: renamed from C46; footprint Capacitor_SMD:C_0603_1608Metric -> Capacitor_SMD:C_0402_1005Metric; KiLib_Generator (none) -> SMD_2terminal_chip_molded
- C46: renamed from C47; footprint Capacitor_SMD:C_0603_1608Metric -> Capacitor_SMD:C_0402_1005Metric; KiLib_Generator (none) -> SMD_2terminal_chip_molded
- R22: renamed from R21; value 1m -> 1M
- renumbered R22 to R25, U13 to U14, U16 to U17
Connections:
- net +3V3: now also C115.1, C116.1, C121.1
- net +3V3A_PCIE: now also C120.1
- net GND: now also C115.2, C116.2, C120.2, C121.2
Other:
- moved on the sheet: FB3

Commit message: Assigned all parts with JLCPCB plugin
Parts:
- C115, C116, C121, C122, C46: LCSC (none) -> C1525
- C120: LCSC (none) -> C1779
- C39, C41: LCSC (none) -> C327316
- C40, C42, C43, C44: LCSC (none) -> C14663
- FB3: LCSC (none) -> C85840
- R22: LCSC (none) -> C22935
- R25: LCSC (none) -> C21189
- Y2: LCSC (none) -> C5742221
Changed lines of the file:
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@@
+			)
+		)
+		(property "LCSC" "C1525"
+			(at 21.59 162.56 0)
+			(hide yes)
+			(show_name no)
+			(do_not_autoplace no)
+			(effects
+				(font
+					(size 1.27 1.27)
+				)
 			)
 		)
@@
 		)
 		(property "KiLib_Generator" "SMD_2terminal_chip_molded"
+			(at 57.15 165.1 0)
+			(hide yes)
+			(show_name no)
+			(do_not_autoplace no)
+			(effects
+				(font
+					(size 1.27 1.27)
+				)
+			)
+		)
+		(property "LCSC" "C1525"
 			(at 57.15 165.1 0)
 			(hide yes)
@@
 			)
 		)
+		(property "LCSC" "C14663"
+			(at 194.31 64.77 0)
+			(hide yes)
+			(show_name no)
+			(do_not_autoplace no)
+			(effects
+				(font
+					(size 1.27 1.27)
+				)
+			)
+		)
 		(pin "1"
 		)
@@
 		)
 		(property "Description" "Resistor"
+			(at 33.02 74.93 0)
+			(hide yes)
+			(show_name no)
+			(do_not_autoplace no)
+			(effects
+				(font
+					(size 1.27 1.27)
+				)
+			)
+		)
+		(property "LCSC" "C22935"
 			(at 33.02 74.93 0)
 			(hide yes)
@@
 			)
 		)
+		(property "LCSC" "C327316"
+			(at 29.21 78.74 0)
+			(hide yes)
+			(show_name no)
+			(do_not_autoplace no)
+			(effects
+				(font
+					(size 1.27 1.27)
+				)
+			)
+		)
 		(pin "2"
 		)
@@
 			)
 		)
+		(property "LCSC" "C85840"
+			(at 46.99 156.21 0)
+			(hide yes)
+			(show_name no)
+			(do_not_autoplace no)
+			(effects
+				(font
+					(size 1.27 1.27)
+				)
+			)
+		)
 		(pin "1"
 		)
@@
 			)
 		)
+		(property "LCSC" "C1525"
+			(at 31.75 162.56 0)
+			(hide yes)
+			(show_name no)
+			(do_not_autoplace no)
+			(effects
+				(font
+					(size 1.27 1.27)
+				)
+			)
+		)
 		(pin "1"
 		)
@@
 		)
 		(property "Description" "Unpolarized capacitor"
+			(at 29.21 71.12 0)
+			(hide yes)
+			(show_name no)
+			(do_not_autoplace no)
+			(effects
+				(font
+					(size 1.27 1.27)
+				)
+			)
+		)
+		(property "LCSC" "C327316"
 			(at 29.21 71.12 0)
 			(hide yes)
@@
 			)
 		)
+		(property "LCSC" "C1779"
+			(at 49.53 165.1 0)
+			(hide yes)
+			(show_name no)
+			(do_not_autoplace no)
+			(effects
+				(font
+					(size 1.27 1.27)
+				)
+			)
+		)
 		(pin "1"
 		)
@@
 			)
 		)
+		(property "LCSC" "C1525"
+			(at 26.67 162.56 0)
+			(hide yes)
+			(show_name no)
+			(do_not_autoplace no)
+			(effects
+				(font
+					(size 1.27 1.27)
+				)
+			)
+		)
 		(pin "1"
 		)
@@
 			)
 		)
+		(property "LCSC" "C14663"
+			(at 130.81 66.04 0)
+			(hide yes)
+			(show_name no)
+			(do_not_autoplace no)
+			(effects
+				(font
+					(size 1.27 1.27)
+				)
+			)
+		)
 		(pin "1"
 		)
@@
 			)
 		)
+		(property "LCSC" "C21189"
+			(at 107.95 73.66 0)
+			(hide yes)
+			(show_name no)
+			(do_not_autoplace no)
+			(effects
+				(font
+					(size 1.27 1.27)
+				)
+			)
+		)
 		(pin "2"
 		)
@@
 			)
 		)
+		(property "LCSC" "C14663"
+			(at 127 63.5 0)
+			(hide yes)
+			(show_name no)
+			(do_not_autoplace no)
+			(effects
+				(font
+					(size 1.27 1.27)
+				)
+			)
+		)
 		(pin "1"
 		)
@@
 			)
 		)
+		(property "LCSC" "C14663"
+			(at 191.77 62.23 0)
+			(hide yes)
+			(show_name no)
+			(do_not_autoplace no)
+			(effects
+				(font
+					(size 1.27 1.27)
+				)
+			)
+		)
 		(pin "1"
 		)
@@
 			)
 		)
+		(property "LCSC" "C1525"
+			(at 36.83 162.56 0)
+			(hide yes)
+			(show_name no)
+			(do_not_autoplace no)
+			(effects
+				(font
+					(size 1.27 1.27)
+				)
+			)
+		)
 		(pin "1"
 		)
@@
 			(at 40.64 74.93 0)
 			(hide yes)
+			(show_name no)
+			(do_not_autoplace no)
+			(effects
+				(font
+					(size 1.27 1.27)
+				)
+			)
+		)
+		(property "LCSC" "C5742221"
+			(at 40.64 74.93 0)
+			(hide yes)

Commit message: Added series resistors to all CT lines. They ring up to 7V apparently according to Super Videl devs. Some of that is likely the length of scope lines. The safety fix here is to add small 33ohm resistors and to enable clamp diodes in the FPGA core.
Parts:
- renumbered R22 to R39, R25 to R44
Changed lines of the file:
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@@
 		(in_pos_files yes)
 		(dnp no)
-		(property "Reference" "R22"
+		(property "Reference" "R39"
 			(at 26.67 75.692 0)
 			(show_name no)
@@
 			(project "mega_videl"
 				(path "/10511203-7d65-4cdf-a1a4-c07b44ea87e2/2e9ae4b7-1d52-4a57-bd5b-5fd3b8f07f63"
-					(reference "R22")
+					(reference "R39")
 					(unit 1)
 				)
@@
 		(dnp yes)
 		(fields_autoplaced yes)
-		(property "Reference" "R25"
+		(property "Reference" "R44"
 			(at 110.49 72.3899 0)
 			(show_name no)
@@
 			(project "mega_videl"
 				(path "/10511203-7d65-4cdf-a1a4-c07b44ea87e2/2e9ae4b7-1d52-4a57-bd5b-5fd3b8f07f63"
-					(reference "R25")
-					(unit 1)
-				)
+					(reference "R44")
+					(unit 1)
+				)
