File: board/kicad/mega_videl/ddr3.kicad_sch (KiCad schematic)
At the start: 14 parts, among them U2 MT41K256M16LY, U3 MT41K256M16LY

Commit message: Reviewed and fixed many issues. e.g. missing decoupling for 1.35v under fpga
Parts:
- R34: renamed from R29; value 2k -> 10k
- U2, U3: LCSC Part (none) -> C20446380
- renumbered R30 to R35, R31 to R36, R32 to R37
Connections:
- net +1V35: no longer R34.1
- net GND: now also R34.1
Changed lines of the file:
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@@
 	)
 	(junction
-		(at 128.27 50.8)
-		(diameter 0)
-		(color 0 0 0 0)
-	)
-	(junction
 		(at 102.87 160.02)
 		(diameter 0)
@@
 	(wire
 		(pts
-			(xy 124.46 50.8) (xy 128.27 50.8)
+			(xy 124.46 50.8) (xy 133.35 50.8)
 		)
 		(stroke
@@
 	(wire
 		(pts
+			(xy 146.05 46.99) (xy 146.05 48.26)
+		)
+		(stroke
+			(width 0)
+			(type default)
+		)
+	)
+	(wire
+		(pts
 			(xy 124.46 48.26) (xy 124.46 50.8)
 		)
@@
 	(wire
 		(pts
-			(xy 128.27 46.99) (xy 128.27 50.8)
-		)
-		(stroke
-			(width 0)
-			(type default)
-		)
-	)
-	(wire
-		(pts
 			(xy 40.64 78.74) (xy 52.07 78.74)
 		)
@@
 	(wire
 		(pts
-			(xy 128.27 50.8) (xy 133.35 50.8)
-		)
-		(stroke
-			(width 0)
-			(type default)
-		)
-	)
-	(wire
-		(pts
 			(xy 102.87 154.94) (xy 102.87 160.02)
 		)
@@
 	(wire
 		(pts
-			(xy 148.59 46.99) (xy 128.27 46.99)
-		)
-		(stroke
-			(width 0)
-			(type default)
-		)
-	)
-	(wire
-		(pts
 			(xy 209.55 55.88) (xy 209.55 58.42)
 		)
@@
 	(wire
 		(pts
+			(xy 148.59 46.99) (xy 146.05 46.99)
+		)
+		(stroke
+			(width 0)
+			(type default)
+		)
+	)
+	(wire
+		(pts
 			(xy 262.89 50.8) (xy 274.32 50.8)
 		)
@@
 		)
 	)
-	(label "unconnected-(RN3-Pad8)"
-		(at 191.77 140.97 180)
-		(effects
-			(font
-				(size 1.27 1.27)
-			)
-			(justify right bottom)
-		)
-	)
 	(label "DRAM.CAS_N"
 		(at 234.95 109.22 0)
@@
 		)
 	)
-	(label "unconnected-(RN7-Pad1)"
-		(at 255.27 99.06 180)
-		(effects
-			(font
-				(size 1.27 1.27)
-			)
-			(justify right bottom)
-		)
-	)
 	(label "DRAM.A7"
 		(at 110.49 78.74 0)
@@
 		(in_pos_files yes)
 		(dnp no)
-		(property "Reference" "R29"
+		(property "Reference" "R34"
 			(at 152.654 46.736 90)
 			(show_name no)
@@
 			)
 		)
-		(property "Value" "2k"
+		(property "Value" "10k"
 			(at 152.654 49.276 90)
 			(show_name no)
@@
 			(project "mega_videl"
 				(path "/10511203-7d65-4cdf-a1a4-c07b44ea87e2/9cd86b33-7f66-43be-a075-05e508a6c489"
-					(reference "R29")
+					(reference "R34")
 					(unit 1)
 				)
@@
 		(dnp no)
 		(fields_autoplaced yes)
-		(property "Reference" "R32"
+		(property "Reference" "R37"
 			(at 185.42 147.3199 0)
 			(show_name no)
@@
 			(project "mega_videl"
 				(path "/10511203-7d65-4cdf-a1a4-c07b44ea87e2/9cd86b33-7f66-43be-a075-05e508a6c489"
-					(reference "R32")
+					(reference "R37")
 					(unit 1)
 				)
@@
 			)
 		)
+		(property "LCSC Part" "C20446380"
+			(at 67.31 101.6 0)
+			(hide yes)
+			(show_name no)
+			(do_not_autoplace no)
+			(effects
+				(font
+					(size 1.27 1.27)
+				)
+			)
+		)
 		(pin "P3"
 		)
@@
 		(dnp no)
 		(fields_autoplaced yes)
-		(property "Reference" "R30"
+		(property "Reference" "R35"
 			(at 156.21 148.5899 0)
 			(show_name no)
@@
 			(project "mega_videl"
 				(path "/10511203-7d65-4cdf-a1a4-c07b44ea87e2/9cd86b33-7f66-43be-a075-05e508a6c489"
-					(reference "R30")
+					(reference "R35")
+					(unit 1)
+				)
+			)
+		)
+	)
+	(symbol
+		(lib_id "power:GND")
+		(at 146.05 48.26 0)
+		(unit 1)
+		(body_style 1)
+		(exclude_from_sim no)
+		(in_bom yes)
+		(on_board yes)
+		(in_pos_files yes)
+		(dnp no)
+		(fields_autoplaced yes)
+		(property "Reference" "#PWR0122"
+			(at 146.05 54.61 0)
+			(hide yes)
+			(show_name no)
+			(do_not_autoplace no)
+			(effects
+				(font
+					(size 1.27 1.27)
+				)
+			)
+		)
+		(property "Value" "GND"
+			(at 146.05 53.34 0)
+			(show_name no)
+			(do_not_autoplace no)
+			(effects
+				(font
+					(size 1.27 1.27)
+				)
+			)
+		)
+		(property "Footprint" ""
+			(at 146.05 48.26 0)
+			(hide yes)
+			(show_name no)
+			(do_not_autoplace no)
+			(effects
+				(font
+					(size 1.27 1.27)
+				)
+			)
+		)
+		(property "Datasheet" ""
+			(at 146.05 48.26 0)
+			(hide yes)
+			(show_name no)
+			(do_not_autoplace no)
+			(effects
+				(font
+					(size 1.27 1.27)
+				)
+			)
+		)
+		(property "Description" "Power symbol creates a global label with name \"GND\" , ground"
+			(at 146.05 48.26 0)
+			(hide yes)
+			(show_name no)
+			(do_not_autoplace no)
+			(effects
+				(font
+					(size 1.27 1.27)
+				)
+			)
+		)
+		(pin "1"
+		)
+		(instances
+			(project "mega_videl"
+				(path "/10511203-7d65-4cdf-a1a4-c07b44ea87e2/9cd86b33-7f66-43be-a075-05e508a6c489"
+					(reference "#PWR0122")
 					(unit 1)
 				)
@@
 		(dnp no)
 		(fields_autoplaced yes)
-		(property "Reference" "R31"
+		(property "Reference" "R36"
 			(at 105.41 149.8599 0)
 			(show_name no)
@@
 			(project "mega_videl"
 				(path "/10511203-7d65-4cdf-a1a4-c07b44ea87e2/9cd86b33-7f66-43be-a075-05e508a6c489"
-					(reference "R31")
+					(reference "R36")
 					(unit 1)
 				)
@@
 			(hide yes)
 			(show_name no)
+			(do_not_autoplace no)
+			(effects
+				(font
+					(size 1.27 1.27)
+				)
+			)
+		)
+		(property "LCSC Part" "C20446380"
+			(at 135.89 101.6 0)
+			(hide yes)
+			(show_name no)

Commit message: Assigned all parts with JLCPCB plugin
Parts:
- R3, R4: LCSC (none) -> C25087
- R34: LCSC (none) -> C25804
- R35, R36: LCSC (none) -> C23350
- R37: LCSC (none) -> C23162
- U2, U3: LCSC Part C20446380 -> C253882
Changed lines of the file:
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@@
+			)
+		)
+		(property "LCSC" "C25804"
+			(at 152.4 46.99 0)
+			(hide yes)
+			(show_name no)
+			(do_not_autoplace no)
+			(effects
+				(font
+					(size 1.27 1.27)
+				)
 			)
 		)
@@
 			)
 		)
+		(property "LCSC" "C23162"
+			(at 182.88 148.59 0)
+			(hide yes)
+			(show_name no)
+			(do_not_autoplace no)
+			(effects
+				(font
+					(size 1.27 1.27)
+				)
+			)
+		)
 		(pin "1"
 		)
@@
 		)
 		(property "KiLib_Generator" "SMD_2terminal_chip_molded"
+			(at 201.93 144.78 0)
+			(hide yes)
+			(show_name no)
+			(do_not_autoplace no)
+			(effects
+				(font
+					(size 1.27 1.27)
+				)
+			)
+		)
+		(property "LCSC" "C25087"
 			(at 201.93 144.78 0)
 			(hide yes)
@@
 			)
 		)
-		(property "LCSC Part" "C20446380"
+		(property "LCSC Part" "C253882"
 			(at 67.31 101.6 0)
 			(hide yes)
@@
 			)
 		)
+		(property "LCSC" "C23350"
+			(at 153.67 149.86 0)
+			(hide yes)
+			(show_name no)
+			(do_not_autoplace no)
+			(effects
+				(font
+					(size 1.27 1.27)
+				)
+			)
+		)
 		(pin "1"
 		)
@@
 			)
 		)
+		(property "LCSC" "C23350"
+			(at 102.87 151.13 0)
+			(hide yes)
+			(show_name no)
+			(do_not_autoplace no)
+			(effects
+				(font
+					(size 1.27 1.27)
+				)
+			)
+		)
 		(pin "1"
 		)
@@
 		)
 		(property "KiLib_Generator" "SMD_2terminal_chip_molded"
+			(at 219.71 144.78 0)
+			(hide yes)
+			(show_name no)
+			(do_not_autoplace no)
+			(effects
+				(font
+					(size 1.27 1.27)
+				)
+			)
+		)
+		(property "LCSC" "C25087"
 			(at 219.71 144.78 0)
 			(hide yes)
@@
 			)
 		)
-		(property "LCSC Part" "C20446380"
+		(property "LCSC Part" "C253882"
 			(at 135.89 101.6 0)
 			(hide yes)

Commit message: Added series resistors to all CT lines. They ring up to 7V apparently according to Super Videl devs. Some of that is likely the length of scope lines. The safety fix here is to add small 33ohm resistors and to enable clamp diodes in the FPGA core.
Parts:
- renumbered R34 to R53, R35 to R54, R36 to R55, R37 to R58
Changed lines of the file:
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@@
 		(in_pos_files yes)
 		(dnp no)
-		(property "Reference" "R34"
+		(property "Reference" "R53"
 			(at 152.654 46.736 90)
 			(show_name no)
@@
 			(project "mega_videl"
 				(path "/10511203-7d65-4cdf-a1a4-c07b44ea87e2/9cd86b33-7f66-43be-a075-05e508a6c489"
-					(reference "R34")
+					(reference "R53")
 					(unit 1)
 				)
@@
 		(dnp no)
 		(fields_autoplaced yes)
-		(property "Reference" "R37"
+		(property "Reference" "R58"
 			(at 185.42 147.3199 0)
 			(show_name no)
@@
 			(project "mega_videl"
 				(path "/10511203-7d65-4cdf-a1a4-c07b44ea87e2/9cd86b33-7f66-43be-a075-05e508a6c489"
-					(reference "R37")
+					(reference "R58")
 					(unit 1)
 				)
@@
 		(dnp no)
 		(fields_autoplaced yes)
-		(property "Reference" "R35"
+		(property "Reference" "R54"
 			(at 156.21 148.5899 0)
 			(show_name no)
@@
 			(project "mega_videl"
 				(path "/10511203-7d65-4cdf-a1a4-c07b44ea87e2/9cd86b33-7f66-43be-a075-05e508a6c489"
-					(reference "R35")
+					(reference "R54")
 					(unit 1)
 				)
@@
 		(dnp no)
 		(fields_autoplaced yes)
-		(property "Reference" "R36"
+		(property "Reference" "R55"
 			(at 105.41 149.8599 0)
 			(show_name no)
@@
 			(project "mega_videl"
 				(path "/10511203-7d65-4cdf-a1a4-c07b44ea87e2/9cd86b33-7f66-43be-a075-05e508a6c489"
-					(reference "R36")
+					(reference "R55")
 					(unit 1)
 				)
