File: board/kicad/mega_videl/usb2.kicad_sch (KiCad schematic)
At the start: 24 parts, among them U10 TXV0108RGYR, U11 USB3300-EZK, U12 AP2553AW6-7, Y1 24MHz

Commit message: Reviewed and fixed many issues. e.g. missing decoupling for 1.35v under fpga
Parts:
- added D3: TPD4E6B06DPWR, mega_videl:X2SON-4_L0.8-W0.8-P0.48-TL-A, symbol mega_videl:TPD4E6B06DPWR
- added R49: 10k, Resistor_SMD:R_0603_1608Metric, symbol Device:R
- C36: value 4.7uF -> 10uF; footprint Capacitor_SMD:C_0603_1608Metric -> Capacitor_SMD:C_0805_2012Metric; KiLib_Generator (none) -> SMD_2terminal_chip_molded
- R16: value 1m -> 1M
- U13: renamed from U12; LCSC Part (none) -> C441827
- renumbered C97 to C106, C104 to C113, C105 to C114, R25 to R30, R26 to R31, U10 to U11, U11 to U12
Connections:
- net +3V3: now also R49.1
- net GND: now also D3.5 (GND)
- net Net-(U20-EXTVBUS): now also R49.2
- net USBD_N: now also D3.2 (IO2)
- net USBD_P: now also D3.3 (IO3)
- net at R31.1, USBC1.B5 (CC2): now also D3.4 (IO4)
- net at R30.1, USBC1.A5 (CC1): now also D3.1 (IO1)

Commit message: Assigned all parts with JLCPCB plugin
Parts:
- C106, C30, C31, C32, C33, C37: LCSC (none) -> C14663
- C113, C114: footprint Capacitor_SMD:C_0603_1608Metric -> Capacitor_SMD:C_0805_2012Metric; KiLib_Generator (none) -> SMD_2terminal_chip_molded; LCSC (none) -> C1779
- C34, C35: value 22pF -> 30pF; LCSC (none) -> C1658
- C36: LCSC (none) -> C15850
- C38: value 120uF -> 100uF; LCSC (none) -> C7432784
- R15: LCSC (none) -> C21189
- R16: LCSC (none) -> C22935
- R17: LCSC (none) -> C23253
- R18: LCSC (none) -> C22790
- R20: LCSC (none) -> C4184
- R30, R31: LCSC (none) -> C23206
- R49: LCSC (none) -> C25804
- U12: LCSC (none) -> C108383
- Y1: LCSC (none) -> C5308006

Commit message: Added series resistors to all CT lines. They ring up to 7V apparently according to Super Videl devs. Some of that is likely the length of scope lines. The safety fix here is to add small 33ohm resistors and to enable clamp diodes in the FPGA core.
Parts:
- renumbered R49 to R123, R15 to R27, R16 to R29, R17 to R30, R18 to R31, R20 to R34, R30 to R49, R31 to R50
Changed lines of the file:
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@@
 		(dnp no)
 		(fields_autoplaced yes)
-		(property "Reference" "R31"
+		(property "Reference" "R50"
 			(at 205.74 137.1599 0)
 			(show_name no)
@@
 			(project "mega_videl"
 				(path "/10511203-7d65-4cdf-a1a4-c07b44ea87e2/4308f970-ce3e-4b29-90b9-8b72e32b0b6e"
-					(reference "R31")
+					(reference "R50")
 					(unit 1)
 				)
@@
 		(dnp no)
 		(fields_autoplaced yes)
-		(property "Reference" "R18"
+		(property "Reference" "R31"
 			(at 152.4 120.6499 0)
 			(show_name no)
@@
 			(project "mega_videl"
 				(path "/10511203-7d65-4cdf-a1a4-c07b44ea87e2/4308f970-ce3e-4b29-90b9-8b72e32b0b6e"
-					(reference "R18")
+					(reference "R31")
 					(unit 1)
 				)
@@
 		(dnp no)
 		(fields_autoplaced yes)
-		(property "Reference" "R17"
+		(property "Reference" "R30"
 			(at 149.86 73.66 90)
 			(show_name no)
@@
 			(project "mega_videl"
 				(path "/10511203-7d65-4cdf-a1a4-c07b44ea87e2/4308f970-ce3e-4b29-90b9-8b72e32b0b6e"
-					(reference "R17")
+					(reference "R30")
 					(unit 1)
 				)
@@
 		(in_pos_files yes)
 		(dnp no)
-		(property "Reference" "R20"
+		(property "Reference" "R34"
 			(at 212.852 70.358 0)
 			(show_name no)
@@
 			(project "mega_videl"
 				(path "/10511203-7d65-4cdf-a1a4-c07b44ea87e2/4308f970-ce3e-4b29-90b9-8b72e32b0b6e"
-					(reference "R20")
+					(reference "R34")
 					(unit 1)
 				)
@@
 		(dnp no)
 		(fields_autoplaced yes)
-		(property "Reference" "R30"
+		(property "Reference" "R49"
 			(at 196.85 137.1599 0)
 			(show_name no)
@@
 			(project "mega_videl"
 				(path "/10511203-7d65-4cdf-a1a4-c07b44ea87e2/4308f970-ce3e-4b29-90b9-8b72e32b0b6e"
-					(reference "R30")
+					(reference "R49")
 					(unit 1)
 				)
@@
 		(in_pos_files yes)
 		(dnp no)
-		(property "Reference" "R16"
+		(property "Reference" "R29"
 			(at 166.37 94.488 0)
 			(show_name no)
@@
 			(project "mega_videl"
 				(path "/10511203-7d65-4cdf-a1a4-c07b44ea87e2/4308f970-ce3e-4b29-90b9-8b72e32b0b6e"
-					(reference "R16")
+					(reference "R29")
 					(unit 1)
 				)
@@
 		(dnp yes)
 		(fields_autoplaced yes)
-		(property "Reference" "R15"
+		(property "Reference" "R27"
 			(at 97.79 121.9199 0)
 			(show_name no)
@@
 			(project "mega_videl"
 				(path "/10511203-7d65-4cdf-a1a4-c07b44ea87e2/4308f970-ce3e-4b29-90b9-8b72e32b0b6e"
-					(reference "R15")
+					(reference "R27")
 					(unit 1)
 				)
@@
 		(in_pos_files yes)
 		(dnp no)
-		(property "Reference" "R49"
+		(property "Reference" "R123"
 			(at 202.692 58.928 0)
 			(show_name no)
@@
 			(project "mega_videl"
 				(path "/10511203-7d65-4cdf-a1a4-c07b44ea87e2/4308f970-ce3e-4b29-90b9-8b72e32b0b6e"
-					(reference "R49")
+					(reference "R123")
 					(unit 1)
 				)
