File: board/kicad/mega_videl/fpga.kicad_sch (KiCad schematic)
At the start: 47 parts, among them J4 FPGA JTAG, U17 CDCBT1001DPWR, U18 M25PX32-VMW, U9 5CFGXFC4F23, Y4 ASE-50MHz

Commit message: Reviewed and fixed many issues. e.g. missing decoupling for 1.35v under fpga
Parts:
- removed C80, C96: 0.1uF, Capacitor_SMD:C_0402_1005Metric, symbol Device:C
- added C79, C82, C86, C89, C91, C92: 0.1uF, Capacitor_SMD:C_0402_1005Metric, symbol Device:C
- added C83, C84: 4.7uF, Capacitor_SMD:C_0805_2012Metric, symbol Device:C
- added R44, R45: 0, Resistor_SMD:R_0402_1005Metric, symbol Device:R
- U10: renamed from U9; value 5CFGXFC4F23 -> 5CGXFC5C6F23I7N
- U10: renamed from U9; value 5CFGXFC4F23 -> 5CGXFC5C6F23I7N; footprint mega_videl:FBGA-484_L23.0-W23.0-R22-C22-P1.00-TL -> cyclonevef23:FBGA-484_L23.0-W23.0-R22-C22-P1.00-TL
- U19: renamed from U18; value M25PX32-VMW -> N25Q/MT25Q
- renumbered C89 to C100, C90 to C101, C91 to C102, C92 to C103, C93 to C104, C94 to C105, C98 to C107, C99 to C108, C100 to C109, C101 to C110, C102 to C111, C103 to C112, C78 to C80, C79 to C85, C81 to C88, C82 to C90, C83 to C93, C84 to C94, C85 to C96, C86 to C97, C87 to C98, C88 to C99, J4 to J3, R33 to R38, R34 to R39, R35 to R40, R36 to R41, R38 to R42, R37 to R43, R39 to R46, R40 to R47, R41 to R48, R42 to R50, U17 to U18
Connections:
- net unconnected-(U5special-AS_DATA2-PadAA5) is gone; now on net Net-(U29-~{W}/V_{PP}): U10.AA5 (AS_DATA2)
- net unconnected-(U5special-AS_DATA3-PadT4) is gone; now on net Net-(U29-~{HOLD}): U10.T4 (AS_DATA3)
- net +1V1_TX: now also C83.1
- net +1V35: now also C95.1, C79.1, C82.1, C91.1, C92.1
- net +2V5: now also C86.1, C89.1; no longer C95.1, R12.1, R39.1, R41.1, U10.F8 (VCCPGM[3]), U10.R19 (VCCPGM[3]), U10.V8 (VCCPGM[3])
- net +2V5_TX: now also C84.1
- net +3V3: now also R12.1, R39.1, R41.1, U10.F8 (VCCPGM[3]), U10.R19 (VCCPGM[3]), U10.V8 (VCCPGM[3]), R44.1; no longer U10.L6 (MSEL0)
- net CT.A19: now also U10.T10 (IO); no longer U10.AB8 (IO)
- net CT.A31: now also U10.AB8 (IO); no longer U10.T10 (IO)
- net CT.D13: now also U10.AA20 (IO); no longer U10.T22 (IO)
- net ETH.A6: now also U10.T22 (IO); no longer U10.AA20 (IO)
- net GND: now also C79.2, C82.2, C83.2, C84.2, C86.2, C89.2, C91.2, C92.2, R45.1
- new net: R44.2, R45.2, U10.L6 (MSEL0)
- no-connect marks 27 -> 25
Other:
- note added: "T22 is nCEO, careful"

Commit message: Assigned all parts with JLCPCB plugin
Parts:
- C100, C101, C102, C103, C104, C105, C107, C108, C109, C110, C111, C112, C79, C80, C82, C85, C86, C88, C89, C91, C92, C93, C94, C95, C96, C97, C98, C99: LCSC (none) -> C1525
- C83, C84: LCSC (none) -> C1779
- C90: footprint Capacitor_SMD:C_0603_1608Metric -> Capacitor_SMD:C_0402_1005Metric; KiLib_Generator (none) -> SMD_2terminal_chip_molded; LCSC (none) -> C15195
- FB1, FB2: LCSC (none) -> C85840
- J3: LCSC (none) -> C2884455
- R12, R13, R14, R39, R41, R46, R48, R50: LCSC (none) -> C25804
- R19: LCSC (none) -> C21190
- R38: LCSC (none) -> C23350
- R40, R42, R43, R47: LCSC (none) -> C23345
- R44, R45: LCSC (none) -> C17168
- R8: LCSC (none) -> C22975
- U10: LCSC Part C1550985 -> C1550726
- U19: LCSC (none) -> C2802705; now in the parts list
- Y4: LCSC (none) -> C5203552

Commit message: Added series resistors to all CT lines. They ring up to 7V apparently according to Super Videl devs. Some of that is likely the length of scope lines. The safety fix here is to add small 33ohm resistors and to enable clamp diodes in the FPGA core.
Parts:
- renumbered R46 to R108, R47 to R113, R8 to R12, R48 to R122, R50 to R127, R12 to R16, R13 to R22, R14 to R25, R19 to R32, R38 to R71, R39 to R76, R40 to R81, R41 to R88, R42 to R92, R43 to R93, R44 to R94, R45 to R98
Changed lines of the file:
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@@
 		(dnp no)
 		(fields_autoplaced yes)
-		(property "Reference" "R13"
+		(property "Reference" "R22"
 			(at 232.41 372.1099 0)
 			(show_name no)
@@
 			(project "mega_videl"
 				(path "/10511203-7d65-4cdf-a1a4-c07b44ea87e2/37efc667-8374-4add-951f-3ec382fdef97"
-					(reference "R13")
+					(reference "R22")
 					(unit 1)
 				)
@@
 		(dnp no)
 		(fields_autoplaced yes)
-		(property "Reference" "R38"
+		(property "Reference" "R71"
 			(at 461.01 71.1199 0)
 			(show_name no)
@@
 			(project "mega_videl"
 				(path "/10511203-7d65-4cdf-a1a4-c07b44ea87e2/37efc667-8374-4add-951f-3ec382fdef97"
-					(reference "R38")
+					(reference "R71")
 					(unit 1)
 				)
@@
 		(in_pos_files yes)
 		(dnp no)
-		(property "Reference" "R47"
+		(property "Reference" "R113"
 			(at 216.916 322.58 90)
 			(show_name no)
@@
 			(project "mega_videl"
 				(path "/10511203-7d65-4cdf-a1a4-c07b44ea87e2/37efc667-8374-4add-951f-3ec382fdef97"
-					(reference "R47")
+					(reference "R113")
 					(unit 1)
 				)
@@
 		(dnp yes)
 		(fields_autoplaced yes)
-		(property "Reference" "R45"
+		(property "Reference" "R98"
 			(at 293.37 300.9899 0)
 			(show_name no)
@@
 			(project "mega_videl"
 				(path "/10511203-7d65-4cdf-a1a4-c07b44ea87e2/37efc667-8374-4add-951f-3ec382fdef97"
-					(reference "R45")
+					(reference "R98")
 					(unit 1)
 				)
@@
 		(dnp no)
 		(fields_autoplaced yes)
-		(property "Reference" "R8"
+		(property "Reference" "R12"
 			(at 66.04 427.9899 0)
 			(show_name no)
@@
 			(project "mega_videl"
 				(path "/10511203-7d65-4cdf-a1a4-c07b44ea87e2/37efc667-8374-4add-951f-3ec382fdef97"
-					(reference "R8")
+					(reference "R12")
 					(unit 1)
 				)
@@
 		(dnp no)
 		(fields_autoplaced yes)
-		(property "Reference" "R44"
+		(property "Reference" "R94"
 			(at 287.02 300.9899 0)
 			(show_name no)
@@
 			(project "mega_videl"
 				(path "/10511203-7d65-4cdf-a1a4-c07b44ea87e2/37efc667-8374-4add-951f-3ec382fdef97"
-					(reference "R44")
+					(reference "R94")
 					(unit 1)
 				)
@@
 		(in_pos_files yes)
 		(dnp no)
-		(property "Reference" "R40"
+		(property "Reference" "R81"
 			(at 551.942 336.55 90)
 			(show_name no)
@@
 			(project "mega_videl"
 				(path "/10511203-7d65-4cdf-a1a4-c07b44ea87e2/37efc667-8374-4add-951f-3ec382fdef97"
-					(reference "R40")
+					(reference "R81")
 					(unit 1)
 				)
@@
 		(in_pos_files yes)
 		(dnp no)
-		(property "Reference" "R50"
+		(property "Reference" "R127"
 			(at 212.09 303.53 90)
 			(show_name no)
@@
 			(project "mega_videl"
 				(path "/10511203-7d65-4cdf-a1a4-c07b44ea87e2/37efc667-8374-4add-951f-3ec382fdef97"
-					(reference "R50")
+					(reference "R127")
 					(unit 1)
 				)
@@
 		(dnp no)
 		(fields_autoplaced yes)
-		(property "Reference" "R46"
+		(property "Reference" "R108"
 			(at 226.06 300.9899 0)
 			(show_name no)
@@
 			(project "mega_videl"
 				(path "/10511203-7d65-4cdf-a1a4-c07b44ea87e2/37efc667-8374-4add-951f-3ec382fdef97"
-					(reference "R46")
+					(reference "R108")
 					(unit 1)
 				)
@@
 		(in_pos_files yes)
 		(dnp no)
-		(property "Reference" "R42"
+		(property "Reference" "R92"
 			(at 517.652 290.83 90)
 			(show_name no)
@@
 			(project "mega_videl"
 				(path "/10511203-7d65-4cdf-a1a4-c07b44ea87e2/37efc667-8374-4add-951f-3ec382fdef97"
-					(reference "R42")
+					(reference "R92")
 					(unit 1)
 				)
@@
 		(dnp no)
 		(fields_autoplaced yes)
-		(property "Reference" "R48"
+		(property "Reference" "R122"
 			(at 233.68 300.9899 0)
 			(show_name no)
@@
 			(project "mega_videl"
 				(path "/10511203-7d65-4cdf-a1a4-c07b44ea87e2/37efc667-8374-4add-951f-3ec382fdef97"
-					(reference "R48")
+					(reference "R122")
 					(unit 1)
 				)
@@
 		(in_pos_files yes)
 		(dnp no)
-		(property "Reference" "R39"
+		(property "Reference" "R76"
 			(at 266.446 342.392 90)
 			(show_name no)
@@
 			(project "mega_videl"
 				(path "/10511203-7d65-4cdf-a1a4-c07b44ea87e2/37efc667-8374-4add-951f-3ec382fdef97"
-					(reference "R39")
+					(reference "R76")
 					(unit 1)
 				)
@@
 		(in_pos_files yes)
 		(dnp no)
-		(property "Reference" "R14"
+		(property "Reference" "R25"
 			(at 220.98 372.618 0)
 			(show_name no)
@@
 			(project "mega_videl"
 				(path "/10511203-7d65-4cdf-a1a4-c07b44ea87e2/37efc667-8374-4add-951f-3ec382fdef97"
-					(reference "R14")
+					(reference "R25")
 					(unit 1)
 				)
@@
 		(dnp no)
 		(fields_autoplaced yes)
-		(property "Reference" "R19"
+		(property "Reference" "R32"
 			(at 223.52 398.7799 0)
 			(show_name no)
@@
 			(project "mega_videl"
 				(path "/10511203-7d65-4cdf-a1a4-c07b44ea87e2/37efc667-8374-4add-951f-3ec382fdef97"
-					(reference "R19")
+					(reference "R32")
 					(unit 1)
 				)
@@
 		(in_pos_files yes)
 		(dnp no)
-		(property "Reference" "R41"
+		(property "Reference" "R88"
 			(at 260.35 335.28 90)
 			(show_name no)
@@
 			(project "mega_videl"
 				(path "/10511203-7d65-4cdf-a1a4-c07b44ea87e2/37efc667-8374-4add-951f-3ec382fdef97"
-					(reference "R41")
+					(reference "R88")
 					(unit 1)
 				)
@@
 		(in_pos_files yes)
 		(dnp no)
-		(property "Reference" "R43"
+		(property "Reference" "R93"
 			(at 517.652 295.91 90)
 			(show_name no)
@@
 			(project "mega_videl"
 				(path "/10511203-7d65-4cdf-a1a4-c07b44ea87e2/37efc667-8374-4add-951f-3ec382fdef97"
-					(reference "R43")
+					(reference "R93")
 					(unit 1)
 				)
@@
 		(in_pos_files yes)
 		(dnp no)
-		(property "Reference" "R12"
+		(property "Reference" "R16"
 			(at 266.446 362.712 90)
 			(show_name no)
@@
 			(project "mega_videl"
 				(path "/10511203-7d65-4cdf-a1a4-c07b44ea87e2/37efc667-8374-4add-951f-3ec382fdef97"
-					(reference "R12")
+					(reference "R16")
 					(unit 1)
 				)

Commit message: Shrunk the dimensions to fit better so it does not hit Q1. Added a notch for the DIMM casing.
Parts:
- J3: LCSC C2884455 -> C17323676
Changed lines of the file:
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@@
 			)
 		)
-		(property "LCSC" "C2884455"
+		(property "LCSC" "C17323676"
 			(at 236.22 388.62 0)
 			(hide yes)
